File: hardware/Thermostat/Thermostat.kicad_pcb (KiCad board)
At the start: 2 copper layers, 109.4 x 76.5 mm, 51 parts, among them J1 Barrel_Jack_Switch, J2 Conn_01x02_Pin, J3 AVR-ISP-6, J4 MainConnectorr, K1 G6E, K2 G6E, K3 G6E, K4 G6E, SW1 12MM, SW2 12MM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

Commit message: WIP
Parts:
- removed D1, D2, D3, D4: LED, LED_SMD:LED_0805_2012Metric
- removed R2, R3, R4, R5: 660, Resistor_SMD:R_0603_1608Metric
- removed S1, S3: 2MS1T1B1M2QES, ThermostatFootprints:2MS1T1B1M2QES
- removed Y2: Crystal_GND23, Crystal:Crystal_SMD_5032-2Pin_5.0x3.2mm
- added C7: C, Capacitor_SMD:C_0603_1608Metric, F.Cu at (198.5, 113.5)
- added SW7: 12MM, ThermostatFootprints:B3F, F.Cu at (153.0, 113.0)
- added SW9: 12MM, ThermostatFootprints:B3F, F.Cu at (135.2, 113.0)
- added Y3: Crystal, Crystal:Crystal_SMD_5032-2Pin_5.0x3.2mm, F.Cu at (185.7, 115.0)
- D5: value SM6T27A -> 1N4007; footprint Diode_SMD:D_SMB -> Diode_THT:D_DO-41_SOD81_P10.16mm_Horizontal
- moved R1 58.1 mm to (204.9, 119.1)
- moved SW5 58.1 mm to (201.0, 119.2)
- moved R6 24.2 mm to (202.0, 109.5)
- moved R7 23.7 mm to (201.5, 107.0)
- moved J3 23.0 mm to (174.5, 109.5)
- moved U2 16.6 mm to (193.5, 112.5), turned to 180 degrees
- moved C9 9.49 mm to (192.0, 118.5), turned to 90 degrees
- moved U6 7.86 mm to (194.5, 118.7)
- moved U8 5.45 mm to (185.0, 108.0)
- moved SW4 3.06 mm to (174.5, 117.9)
- moved J2 2.50 mm to (195.0, 106.0), turned to -90 degrees
Connections:
- D5 pad 2: GND -> Net-(D5-A)
- J1 pad 1: 24VDC -> Net-(D5-A)
- K1 pad 1: Net-(U3-OUT1) -> Net-(U3-OUT4)
- K2 pad 1: Net-(U3-OUT2) -> Net-(U3-OUT3)
- K3 pad 1: Net-(U3-OUT3) -> Net-(U3-OUT2)
- K4 pad 1: Net-(U3-OUT4) -> Net-(U3-OUT1)
- SW3 pad 1: Net-(U5-PD7) -> Net-(U5-PD5)
- U1 pad 6: ^RESET -> +5V
- U2 pad 1: unconnected-(U2-VCAP-Pad1) -> Net-(U2-VCAP)
- U2 pad 2: unconnected-(U2-A1-Pad2) -> GND
- U2 pad 3: unconnected-(U2-A2-Pad3) -> GND
- U2 pad 4: unconnected-(U2-VSS-Pad4) -> GND
- U2 pad 5: unconnected-(U2-SDA-Pad5) -> I2C_SDA
- U2 pad 6: unconnected-(U2-SCL-Pad6) -> I2C_SCL
- U2 pad 8: unconnected-(U2-VCC-Pad8) -> +5V
- U5 pad 2: Net-(S1-NC) -> unconnected-(U5-PD4-Pad2)
- U5 pad 9: Net-(S1-NO) -> Net-(U5-PD5)
Routing:
- net Net-(U5-PD6): track 0.00 -> 69.8 mm, vias 0 -> 4
- net I2C_SCL: track 0.00 -> 67.0 mm, vias 0 -> 4
- net I2C_SDA: track 0.00 -> 66.9 mm, vias 0 -> 6
- net Net-(U5-PD7): track 12.5 -> 56.9 mm, vias 0 -> 4
- net SCREEN_BUSY: track 0.00 -> 42.1 mm, vias 0 -> 2
- net Net-(U3-OUT4): track 5.77 -> 43.0 mm
- net Net-(U3-OUT1): track 40.6 -> 5.48 mm
- net +5V: track 6.94 -> 37.6 mm, vias 0 -> 2
- net Net-(J3-MOSI): track 0.00 -> 30.3 mm, vias 0 -> 2
- net GND: track 122.6 -> 152.8 mm
- net ^RESET: track 0.00 -> 28.2 mm, vias 0 -> 4
- net Net-(J3-SCK): track 0.00 -> 25.0 mm, vias 0 -> 2
- net Net-(J3-MISO): track 0.00 -> 24.9 mm
- net Net-(U5-PC3): track 0.00 -> 19.8 mm, vias 0 -> 2
- net Net-(U3-OUT3): track 15.9 -> 29.5 mm
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Other:
- board text removed: "G6E"

Commit message: WIP
Routing:
- net Net-(U5-PD5): track 12.5 -> 42.8 mm, vias 0 -> 2
- net GND: track 152.8 -> 160.1 mm, vias 0 -> 2
Changed lines of the file:
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@@
+	)
+	(segment
+		(start 183.6961 99.0059)
+		(end 184.15 98.552)
+		(width 0.6)
+		(layer "F.Cu")
+		(net 1)
+	)
+	(segment
+		(start 189 98.2299)
+		(end 188.976 98.2059)
+		(width 0.5)
+		(layer "F.Cu")
+		(net 1)
 	)
 	(segment
@@
 	)
 	(segment
-		(start 189 98.5)
-		(end 189 99.5)
-		(width 0.5)
-		(layer "F.Cu")
-		(net 1)
-	)
-	(segment
 		(start 194.405 97.5)
 		(end 198 97.5)
@@
 	)
 	(segment
-		(start 190.4781 98.2059)
-		(end 189.2941 98.2059)
-		(width 0.5)
-		(layer "F.Cu")
-		(net 1)
-	)
-	(segment
 		(start 172.212 115.062)
 		(end 172.212 116.777)
@@
 	)
 	(segment
-		(start 189.2941 98.2059)
-		(end 189 98.5)
-		(width 0.5)
-		(layer "F.Cu")
-		(net 1)
-	)
-	(segment
 		(start 180.594 97.320714)
 		(end 180.594 99.0059)
@@
 		(start 180.594 99.0059)
 		(end 182.1531 99.0059)
+		(width 0.6)
+		(layer "F.Cu")
+		(net 1)
+	)
+	(segment
+		(start 188.976 98.2059)
+		(end 190.4781 98.2059)
 		(width 0.6)
 		(layer "F.Cu")
@@
 	)
 	(segment
+		(start 182.1531 99.0059)
+		(end 183.6961 99.0059)
+		(width 0.6)
+		(layer "F.Cu")
+		(net 1)
+	)
+	(segment
 		(start 189.3059 99.8059)
 		(end 190.4781 99.8059)
@@
 	)
 	(segment
+		(start 188.214 98.2059)
+		(end 188.976 98.2059)
+		(width 0.6)
+		(layer "F.Cu")
+		(net 1)
+	)
+	(segment
 		(start 198.5 88.5)
 		(end 198.349 88.651)
+		(width 0.5)
+		(layer "F.Cu")
+		(net 1)
+	)
+	(segment
+		(start 189 99.5)
+		(end 189 98.2299)
 		(width 0.5)
 		(layer "F.Cu")
@@
 		(net 1)
 	)
+	(via
+		(at 188.214 98.2059)
+		(size 0.6)
+		(drill 0.3)
+		(layers "F.Cu" "B.Cu")
+		(net 1)
+	)
+	(via
+		(at 184.15 98.552)
+		(size 0.6)
+		(drill 0.3)
+		(layers "F.Cu" "B.Cu")
+		(net 1)
+	)
+	(segment
+		(start 186.436 98.552)
+		(end 184.15 98.552)
+		(width 0.6)
+		(layer "B.Cu")
+		(net 1)
+	)
+	(segment
+		(start 186.7821 98.2059)
+		(end 186.436 98.552)
+		(width 0.6)
+		(layer "B.Cu")
+		(net 1)
+	)
+	(segment
+		(start 188.214 98.2059)
+		(end 186.7821 98.2059)
+		(width 0.6)
+		(layer "B.Cu")
+		(net 1)
+	)
 	(segment
 		(start 168.992 94.742)
@@
 	)
 	(segment
-		(start 219.964 105.49)
-		(end 207.464 105.49)
-		(width 0.4)
+		(start 207.464 105.49)
+		(end 202.812 100.838)
+		(width 0.5)
 		(layer "F.Cu")
 		(net 54)
 	)
+	(segment
+		(start 196.596 100.838)
+		(end 195.326 102.108)
+		(width 0.5)
+		(layer "F.Cu")
+		(net 54)
+	)
+	(segment
+		(start 187.198 100.584)
+		(end 187.198 98.044)
+		(width 0.5)
+		(layer "F.Cu")
+		(net 54)
+	)
+	(segment
+		(start 207.464 105.49)
+		(end 219.964 105.49)
+		(width 0.5)
+		(layer "F.Cu")
+		(net 54)
+	)
+	(segment
+		(start 202.692 100.838)
+		(end 196.596 100.838)
+		(width 0.5)
+		(layer "F.Cu")
+		(net 54)
+	)
+	(segment
+		(start 187.198 98.044)
+		(end 189.1156 96.1264)
+		(width 0.5)
+		(layer "F.Cu")
+		(net 54)
+	)
+	(segment
+		(start 189.1156 96.1264)
+		(end 189.1156 94.4434)
+		(width 0.5)
+		(layer "F.Cu")
+		(net 54)
+	)
+	(segment
+		(start 202.812 100.838)
+		(end 202.692 100.838)
+		(width 0.5)
+		(layer "F.Cu")
+		(net 54)
+	)
+	(via
+		(at 187.198 100.584)
+		(size 0.6)
+		(drill 0.3)
+		(layers "F.Cu" "B.Cu")
+		(net 54)
+	)
+	(via
+		(at 195.326 102.108)
+		(size 0.6)
+		(drill 0.3)
+		(layers "F.Cu" "B.Cu")
+		(net 54)
+	)
+	(segment
+		(start 195.326 102.108)
+		(end 188.722 102.108)
+		(width 0.5)
+		(layer "B.Cu")
+		(net 54)
+	)
+	(segment
+		(start 188.722 102.108)
+		(end 187.198 100.584)
+		(width 0.5)
+		(layer "B.Cu")
+		(net 54)
+	)

Commit message: Inching closer and closer
Parts:
- moved R7 13.6 mm to (191.8, 116.5)
- moved D5 12.8 mm to (210.0, 53.4), turned to -90 degrees
- moved R6 9.78 mm to (195.2, 116.5), turned to 180 degrees
- moved C9 1.40 mm to (192.0, 119.9)
- moved U6 1.40 mm to (194.5, 120.1)
- moved Y3 0.65 mm to (185.0, 115.0)
- moved J2 0.50 mm to (195.0, 105.5)
Routing:
- net +5V: track 37.6 -> 114.7 mm, vias 2 -> 5
- net GND: track 160.1 -> 180.2 mm, vias 2 -> 6
- net Net-(U5-PD2): track 21.4 -> 33.9 mm
- net I2C_SDA: track 66.9 -> 75.4 mm
- net I2C_SCL: track 67.0 -> 73.4 mm
- net Net-(U5-PD3): track 48.3 -> 51.6 mm
- net Net-(U2-VCAP): track 0.00 -> 2.58 mm
- net Net-(U5-PD5): track 42.8 -> 41.7 mm

Commit message: WIP
Routing:
- net GND: track 180.2 -> 197.6 mm
- net 24VDC: track 163.3 -> 154.0 mm
Changed lines of the file:
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@@
+	)
+	(segment
+		(start 196.5 88)
+		(end 196.5 84.5)
+		(width 0.5)
+		(layer "F.Cu")
+		(net 1)
 	)
 	(segment
@@
 	)
 	(segment
+		(start 199 90.5)
+		(end 196.5 88)
+		(width 0.5)
+		(layer "F.Cu")
+		(net 1)
+	)
+	(segment
 		(start 199 92)
 		(end 198.5 92.5)
@@
 	)
 	(segment
+		(start 196.5 81.5)
+		(end 201 81.5)
+		(width 0.5)
+		(layer "F.Cu")
+		(net 1)
+	)
+	(segment
 		(start 182.1531 99.0059)
 		(end 183.6961 99.0059)
@@
 	)
 	(segment
+		(start 201 81.5)
+		(end 202 80.5)
+		(width 0.5)
+		(layer "F.Cu")
+		(net 1)
+	)
+	(segment
+		(start 199 92)
+		(end 199 90.5)
+		(width 0.5)
+		(layer "F.Cu")
+		(net 1)
+	)
+	(segment
 		(start 189 99.5)
 		(end 189 98.2299)
@@
 		(end 198.5 111)
 		(width 0.6)
+		(layer "F.Cu")
+		(net 1)
+	)
+	(segment
+		(start 196.5 84.5)
+		(end 196.5 81.5)
+		(width 0.5)
 		(layer "F.Cu")
 		(net 1)
@@
 	)
 	(segment
-		(start 201.831923 75.898)
-		(end 211.487923 66.242)
-		(width 1.5)
-		(layer "F.Cu")
-		(net 2)
-	)
-	(segment
 		(start 182.5 80)
 		(end 182.5 86.5)
@@
 	)
 	(segment
-		(start 177.5 75.898)
-		(end 201.831923 75.898)
-		(width 1.5)
-		(layer "F.Cu")
-		(net 2)
-	)
-	(segment
 		(start 157.75 95)
 		(end 155.2575 92.5075)
@@
 	)
 	(segment
+		(start 177.5 75.898)
+		(end 197.102 75.898)
+		(width 1.5)
+		(layer "F.Cu")
+		(net 2)
+	)
+	(segment
 		(start 166.7575 92.5075)
 		(end 164.265 95)
@@
 		(width 1.5)
 		(layer "F.Cu")
+		(net 2)
+	)
+	(segment
+		(start 197.102 75.898)
+		(end 203.5 69.5)
+		(width 1.5)
+		(layer "F.Cu")

Commit message: WIP
Parts:
- removed U6: TMP116xxDRV, Package_SON:WSON-6-1EP_2x2mm_P0.65mm_EP1x1.6mm_ThermalVias
- added C10: 0.1uF, Capacitor_SMD:C_0603_1608Metric, F.Cu at (191.5, 106.7)
- added C8: 0.1uF, Capacitor_SMD:C_0603_1608Metric, F.Cu at (193.5, 122.2)
- added U9: SHT4x, Sensor_Humidity:Sensirion_DFN-4_1.5x1.5mm_P0.8mm_SHT4x_NoCentralPad, F.Cu at (193.5, 120.0)
- C7: value C -> 6.8uF
- moved R1 24.4 mm to (180.6, 120.4), turned to -90 degrees
- moved SW5 16.4 mm to (184.7, 120.4), turned to 180 degrees
- moved C9 4.30 mm to (189.0, 116.8)
- moved J2 1.09 mm to (196.1, 105.5)
- moved Y3 0.35 mm to (184.7, 115.1)
Connections:
- C9 pad 1: +5V -> GND
- C9 pad 2: GND -> +5V
Routing:
- net GND: track 197.6 -> 253.2 mm, vias 6 -> 7
- net +5V: track 114.7 -> 143.8 mm, vias 5 -> 7
- net ^RESET: track 28.2 -> 51.3 mm, vias 4 -> 6
- net TX0: track 9.06 -> 13.4 mm
- net I2C_SCL: track 73.4 -> 76.3 mm
- net I2C_SDA: track 75.4 -> 78.3 mm
- net RX0: track 9.95 -> 11.9 mm
Other:
- board text removed: "RESET"

Commit message: Wiring / DRC / JLCPCB
Parts:
- C1, C2, C3: footprint Capacitor_SMD:C_0603_1608Metric -> Capacitor_SMD:C_1808_4520Metric
- U5: value ATmega88-20A -> ATmega168P-20A
- moved C1 13.3 mm to (211.8, 54.6), turned to 90 degrees
- moved SW9 12.0 mm to (123.3, 113.3)
- moved SW7 12.0 mm to (141.1, 113.3)
- moved C2 10.6 mm to (215.1, 54.6), turned to 90 degrees
- moved C3 6.15 mm to (213.9, 68.1), turned to 0 degrees
- moved D5 4.93 mm to (206.5, 56.9)
- moved U4 4.88 mm to (214.9, 62.0)
- moved H7 2.08 mm to (118.6, 120.9)
- moved H6 1.52 mm to (118.6, 51.7)
- moved J1 0.71 mm to (130.4, 75.2)
Connections:
- net SCREEN_BUSY renamed SCBUSY
- U5 pad 14: unconnected-(U5-PB2-Pad14) -> Net-(U3-IN4)
- U5 pad 22: Net-(U3-IN4) -> unconnected-(U5-ADC7-Pad22)
Routing:
- net GND: track 253.2 -> 476.0 mm, vias 7 -> 11
- net Net-(D5-A): track 0.00 -> 81.6 mm
- net +5V: track 143.8 -> 189.7 mm, vias 7 -> 9
- net 24VDC: track 154.0 -> 126.3 mm
- net Net-(U5-PD6): track 69.8 -> 81.9 mm
- net Net-(U3-IN4): track 5.65 -> 13.7 mm, vias 0 -> 2
- net Net-(U5-PD7): track 56.9 -> 62.1 mm
- net TX0: track 13.4 -> 10.5 mm
- net Net-(U3-IN1): track 9.98 -> 7.47 mm
- net Net-(U5-PD5): track 41.7 -> 40.9 mm
- net I2C_SCL: track 76.3 -> 76.8 mm
- added copper zone on F.Cu, net GND
Other:
- board size 109.4 x 76.5 mm -> 111.2 x 76.5 mm

Commit message: Some labels
Changed lines of the file:
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@@
 	)
 	(gr_text "FAN"
-		(at 141.05 124.236 0)
+		(at 123 124 0)
 		(layer "F.SilkS")
 		(effects
@@
 	)
 	(gr_text "HEAT"
-		(at 123.05 124.236 0)
+		(at 140.75 123.75 0)
 		(layer "F.SilkS")
 		(effects
@@
 	)
 	(segment
+		(start 189.738 55.552)
+		(end 190.083 55.207)
+		(width 0.5)
+		(layer "F.Cu")
+		(net 26)
+	)
+	(segment
 		(start 185.9156 80.0844)
 		(end 185.9156 94.4434)
@@
 		(width 0.5)
 		(layer "F.Cu")
-		(net 26)
-	)
-	(segment
-		(start 189.738 55.552)
-		(end 190.083 55.207)
-		(width 0.5)
-		(layer "F.Cu")

Commit message: WIP
Parts:
- moved J2 0.25 mm to (196.1, 105.8)
Changed lines of the file:
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@@
 	(footprint "Connector_PinHeader_2.54mm:PinHeader_1x02_P2.54mm_Vertical_SMD_Pin1Left"
 		(layer "F.Cu")
-		(at 196.088 105.5 -90)
+		(at 196.088 105.75 -90)
 		(descr "surface-mounted straight pin header, 1x02, 2.54mm pitch, single row, style 1 (pin 1 left)")
 		(tags "Surface mounted pin header SMD 1x02 2.54mm single row style1 pin1 left")
@@
 	)
 	(segment
-		(start 182.1531 96.6059)
-		(end 181.308814 96.6059)
-		(width 0.6)
-		(layer "F.Cu")
-		(net 1)
-	)
-	(segment
 		(start 172.212 116.777)
 		(end 171.133 117.856)
@@
 	)
 	(segment
-		(start 177.025 112.04)
-		(end 177.025 112.789)
+		(start 182.1531 99.0059)
+		(end 182.1531 98.2059)
 		(width 0.6)
 		(layer "F.Cu")
@@
 	)
 	(segment
-		(start 181.5 112)
-		(end 180.34 112)
+		(start 177.025 112.04)
+		(end 177.025 112.789)
 		(width 0.6)
 		(layer "F.Cu")
@@
 	)
 	(segment
-		(start 181.308814 96.6059)
-		(end 180.594 97.320714)
+		(start 181.5 112)
+		(end 180.34 112)
 		(width 0.6)
 		(layer "F.Cu")
@@
 	)
 	(segment
+		(start 180.8941 96.6059)
+		(end 180.594 96.906)
+		(width 0.6)
+		(layer "F.Cu")
+		(net 1)
+	)
+	(segment
 		(start 219.964 80.732)
 		(end 207.464 80.732)
@@
 	)
 	(segment
+		(start 135.278 72.136)
+		(end 135.23 72.184)
+		(width 1.5)
+		(layer "F.Cu")
+		(net 1)
+	)
+	(segment
 		(start 141.05 121.096)
 		(end 141.05 118.284)
@@
 	)
 	(segment
-		(start 182.1531 98.2059)
-		(end 182.1531 99.0059)
-		(width 0.6)
-		(layer "F.Cu")
-		(net 1)
-	)
-	(segment
 		(start 153.55 117.45)
 		(end 153.55 118.284)
@@
 	)
 	(segment
+		(start 139.192 72.136)
+		(end 135.278 72.136)
+		(width 1.5)
+		(layer "F.Cu")
+		(net 1)
+	)
+	(segment
 		(start 207.464 110.49)
 		(end 219.964 110.49)
@@
 	)
 	(segment
-		(start 180.594 97.320714)
-		(end 180.594 99.0059)
-		(width 0.6)
-		(layer "F.Cu")
-		(net 1)
-	)
-	(segment
 		(start 211.734 61.976)
 		(end 218.034 61.976)
@@
 	)
 	(segment
+		(start 180.594 96.906)
+		(end 180.594 99.0059)
+		(width 0.6)
+		(layer "F.Cu")
+		(net 1)
+	)
+	(segment
 		(start 219.964 90.504)
 		(end 219.964 80.732)
@@
 		(net 1)
 	)
+	(segment
+		(start 182.1531 96.6059)
+		(end 180.8941 96.6059)
+		(width 0.6)
+		(layer "F.Cu")
+		(net 1)
+	)
 	(via
 		(at 205 92)
@@
 	)
 	(segment
-		(start 135.23 72.184)
-		(end 139.144 72.184)
-		(width 1.5)
-		(layer "B.Cu")
-		(net 1)
-	)
-	(segment
 		(start 199 92)
 		(end 205 92)
@@
 	)
 	(segment
-		(start 179.5 96.937926)
-		(end 179.5 98)
+		(start 182.1531 95.8059)
+		(end 179.9441 95.8059)
 		(width 0.5)
 		(layer "F.Cu")
@@
 	)
 	(segment
-		(start 182.1531 95.8059)
-		(end 180.632026 95.8059)
+		(start 179.5 96.25)
+		(end 179.5 98)
 		(width 0.5)
 		(layer "F.Cu")
@@
 	)
 	(segment
-		(start 180.632026 95.8059)
-		(end 179.5 96.937926)
+		(start 179.9441 95.8059)
+		(end 179.5 96.25)
 		(width 0.5)
 		(layer "F.Cu")
@@
 		(polygon
 			(pts
-				(xy 214.884 64.77) (xy 214.884 59.182) (xy 221.488 59.182) (xy 221.488 64.77)
+				(xy 213.884 64.77) (xy 213.884 59.182) (xy 221.488 59.182) (xy 221.488 64.77)
 			)
 		)
 	)
 	(zone
-		(net 9)
-		(net_name "Net-(U3-OUT4)")
+		(net 8)
+		(net_name "Net-(U3-OUT3)")
 		(layer "F.Cu")
 		(name "$teardrop_padvia$")
 		(hatch none 0.1)
-		(priority 30001)
+		(priority 30000)
 		(attr
 			(teardrop
@@
 		(polygon
 			(pts
-				(xy 133.715579 104.102974) (xy 133.362026 103.749421) (xy 131.946603 104.45693) (xy 132.256793 105.208207)
-				(xy 133.00807 105.518396)
+				(xy 145.215579 104.102974) (xy 144.862026 103.749421) (xy 143.446603 104.45693) (xy 143.756793 105.208207)
+				(xy 144.50807 105.518396)
 			)
 		)
@@
 	)
 	(zone
-		(net 8)
-		(net_name "Net-(U3-OUT3)")
+		(net 9)
+		(net_name "Net-(U3-OUT4)")
 		(layer "F.Cu")
 		(name "$teardrop_padvia$")
 		(hatch none 0.1)
-		(priority 30000)
+		(priority 30001)
 		(attr
 			(teardrop
@@
 		(polygon
 			(pts
-				(xy 145.215579 104.102974) (xy 144.862026 103.749421) (xy 143.446603 104.45693) (xy 143.756793 105.208207)
-				(xy 144.50807 105.518396)
+				(xy 133.715579 104.102974) (xy 133.362026 103.749421) (xy 131.946603 104.45693) (xy 132.256793 105.208207)
+				(xy 133.00807 105.518396)
 			)
 		)
